File: schematic/lohpi.kicad_pcb (KiCad board)
At the start: 4 copper layers, 65 x 56 mm, 208 parts, among them J1 CONN_01X02, J10 CONN_01X01, J11 CONN_01X01, J12 CONN_01X01, J13 CONN_01X01, J2 CONN_01X01, J3 CONN_01X01, J4 CONN_01X01, J5 CONN_01X01, J6 CONN_01X01, J7 UFL, J8 raspberry_pi_3_header, J9 CONN_01X02, Q1 Q_PMOS_GSD, U1 MCP1726-3302E/SN, U10 Anaren_B0430J50100AHF, U11 MurataSF2314E, U12 MurataSF2314E, U13 SPF5043Z, U14 RFPA0133TR7, U15 MurataSF2314E, U16 RFSW1012, U17 MurataSF2314E, U18 MAX-M8, U2 MCP1612, U3 MCP1726-3302E/SN, U4 MCP1824, U5 MCP1824, U6 MCP1824, U7 SX1301, U8 SX1257, U9 SX1257, X1 ABRACON-OSC, X2 ABRACON-OSC

Commit message: Correct component for SMPS inductor, changed footprint
Parts:
- L1: footprint Inductors_SMD:L_0805 -> 84332C:84332C
- moved R29 16.6 mm to (108.3, 123.2), turned to 270 degrees
- moved R8 5.91 mm to (135.2, 119.9), turned to 90 degrees
- moved R2 4.95 mm to (144.9, 120.1), turned to 90 degrees
- moved R5 4.35 mm to (144.4, 122.4)
- moved U2 4.35 mm to (139.4, 121.7)
- moved R7 3.74 mm to (132.3, 119.4)
- moved R1 3.56 mm to (140.7, 124.9)
- moved C4 3.53 mm to (146.6, 120.1), turned to 270 degrees
- moved C10 3.50 mm to (143.6, 124.3)
- moved L1 2.16 mm to (131.2, 122.2), turned to 0 degrees
- moved C29 0.45 mm to (129.3, 126.7)
- moved C8 0.39 mm to (129.3, 125.1)
- moved C18 0.28 mm to (125.7, 120.3)
- moved R15 0.13 mm to (124.3, 120.3)
Connections:
- J10 pad 1: Net-(J10-Pad1) -> (no net)
- J11 pad 1: Net-(J11-Pad1) -> (no net)
- J12 pad 1: Net-(J12-Pad1) -> (no net)
- J13 pad 1: Net-(J13-Pad1) -> (no net)
- J8 pad 1: (no net) -> Net-(J8-Pad1)
- J8 pad 16: (no net) -> Net-(J8-Pad16)
- J8 pad 17: (no net) -> Net-(J8-Pad17)
- J8 pad 18: (no net) -> Net-(J8-Pad18)
- J8 pad 22: (no net) -> Net-(J8-Pad22)
- J8 pad 24: (no net) -> Net-(J8-Pad24)
- J8 pad 26: (no net) -> Net-(J8-Pad26)
- J8 pad 27: (no net) -> Net-(J8-Pad27)
- J8 pad 28: (no net) -> Net-(J8-Pad28)
- J8 pad 3: (no net) -> Net-(J8-Pad3)
- J8 pad 32: (no net) -> Net-(J8-Pad32)
- J8 pad 33: (no net) -> Net-(J8-Pad33)
- J8 pad 35: (no net) -> Net-(J8-Pad35)
- J8 pad 36: (no net) -> Net-(J8-Pad36)
- J8 pad 37: (no net) -> Net-(J8-Pad37)
- J8 pad 38: (no net) -> Net-(J8-Pad38)
- J8 pad 40: (no net) -> Net-(J8-Pad40)
- J8 pad 5: (no net) -> Net-(J8-Pad5)
- J8 pad 7: (no net) -> Net-(J8-Pad7)
- U1 pad 5: (no net) -> Net-(U1-Pad5)
- U10 pad 5: Net-(U10-Pad5) -> (no net)
- U14 pad 1: Net-(U14-Pad1) -> (no net)
- U14 pad 11: Net-(U14-Pad11) -> (no net)
- U14 pad 15: Net-(U14-Pad15) -> (no net)
- U14 pad 4: Net-(U14-Pad4) -> (no net)
- U14 pad 5: Net-(U14-Pad5) -> (no net)
- U14 pad 7: Net-(U14-Pad7) -> (no net)
- U14 pad 8: Net-(U14-Pad8) -> (no net)
- U18 pad 13: (no net) -> Net-(U18-Pad13)
- U18 pad 15: (no net) -> Net-(U18-Pad15)
- U18 pad 16: (no net) -> Net-(U18-Pad16)
- U18 pad 17: (no net) -> Net-(U18-Pad17)
- U18 pad 18: (no net) -> Net-(U18-Pad18)
- U18 pad 5: (no net) -> Net-(U18-Pad5)
- U18 pad 9: (no net) -> Net-(U18-Pad9)
- U3 pad 5: (no net) -> Net-(U3-Pad5)
- U4 pad 4: (no net) -> Net-(U4-Pad4)
- U5 pad 4: (no net) -> Net-(U5-Pad4)
- U6 pad 4: (no net) -> Net-(U6-Pad4)
- U7 pad 26: (no net) -> Net-(U7-Pad26)
- U7 pad 27: (no net) -> Net-(U7-Pad27)
- U7 pad 37: (no net) -> Net-(U7-Pad37)
- U7 pad 38: (no net) -> Net-(U7-Pad38)
- U7 pad 54: /main_receiver/GPIO[4] -> (no net)
- U8 pad 11: (no net) -> Net-(U8-Pad11)
- U8 pad 21: (no net) -> Net-(U8-Pad21)
- U8 pad 22: (no net) -> Net-(U8-Pad22)
- U8 pad 23: (no net) -> Net-(U8-Pad23)
- U8 pad 24: (no net) -> Net-(U8-Pad24)
- U8 pad 29: (no net) -> Net-(U8-Pad29)
- U8 pad 30: (no net) -> Net-(U8-Pad30)
- U8 pad 6: (no net) -> Net-(U8-Pad6)
- U9 pad 21: (no net) -> Net-(U9-Pad21)
- U9 pad 22: (no net) -> Net-(U9-Pad22)
- U9 pad 23: (no net) -> Net-(U9-Pad23)
- U9 pad 24: (no net) -> Net-(U9-Pad24)
- U9 pad 6: (no net) -> Net-(U9-Pad6)
- X2 pad 1: Net-(X2-Pad1) -> (no net)
Routing:
- net /main_receiver/A_Q_TX: track 30.4 -> 48.7 mm
- net Net-(R29-Pad2): track 19.4 -> 1.96 mm
- net +1V8: track 86.3 -> 91.5 mm
- net Net-(C3-Pad1): track 5.71 -> 9.53 mm
- net +5V: track 39.2 -> 37.4 mm, vias 6 -> 5
- net GND: track 770.2 -> 772.0 mm, vias 360 -> 359
- net /main_receiver/RPI_5v: track 53.9 -> 55.4 mm
- net Net-(R7-Pad2): track 6.11 -> 4.71 mm
- net Net-(R2-Pad1): track 2.02 -> 3.32 mm
- net Net-(L1-Pad1): track 5.62 -> 4.71 mm

Commit message: Moved all references to F.Fab, cleaned up silkscreen
Parts:
- added J14: CONN_01X01, Pin_Headers:Pin_Header_Straight_1x01_Pitch2.54mm, F.Cu at (149.7, 132.7)
Other:
- board text added: "3.3v"
- board text added: "Gnd"
- board text added: "Radio A"
- board text added: "Vcc LNA_A"
- board text added: "Vcc Radio_B"
- board text added: "Vcc_PA"

Commit message: Version sent to fab
Routing:
- net GND: track 772.0 -> 786.4 mm, vias 359 -> 370
Changed lines of the file:
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@@
-(kicad_pcb (version 20170922) (host pcbnew no-vcs-found-e0b9a21~60~ubuntu16.04.1)
+(kicad_pcb (version 20170922) (host pcbnew no-vcs-found-1929727~60~ubuntu16.04.1)
 (general
   (thickness 1.6)
   (drawings 14)
-  (tracks 2420)
+  (tracks 2452)
   (zones 0)
   (modules 209)
@@
 (layers
   (0 F.Cu signal)
-  (1 In1.Cu power hide)
-  (2 In2.Cu power hide)
-  (31 B.Cu signal hide)
+  (1 In1.Cu power)
+  (2 In2.Cu power)
+  (31 B.Cu signal)
   (32 B.Adhes user)
-  (33 F.Adhes user hide)
+  (33 F.Adhes user)
   (34 B.Paste user)
   (35 F.Paste user)
@@
   (40 Dwgs.User user)
   (41 Cmts.User user)
-  (42 Eco1.User user)
-  (43 Eco2.User user)
+  (42 Eco1.User user hide)
+  (43 Eco2.User user hide)
   (44 Edge.Cuts user)
-  (45 Margin user)
+  (45 Margin user hide)
   (46 B.CrtYd user hide)
   (47 F.CrtYd user hide)
-  (48 B.Fab user)
-  (49 F.Fab user)
-)
-(general
-  (thickness 1.6)
-  (drawings 14)
-  (tracks 2420)
-  (zones 0)
-  (modules 209)
-  (nets 198)
-)
-(page A4)
-(layers
-  (0 F.Cu signal)
-  (1 In1.Cu power hide)
-  (2 In2.Cu power hide)
-  (31 B.Cu signal hide)
-  (32 B.Adhes user)
-  (33 F.Adhes user hide)
-  (34 B.Paste user)
-  (35 F.Paste user)
-  (36 B.SilkS user)
-  (37 F.SilkS user)
-  (38 B.Mask user)
-  (39 F.Mask user)
-  (40 Dwgs.User user)
-  (41 Cmts.User user)
-  (42 Eco1.User user)
-  (43 Eco2.User user)
-  (44 Edge.Cuts user)
-  (45 Margin user)
-  (46 B.CrtYd user hide)
-  (47 F.CrtYd user hide)
-  (48 B.Fab user)
+  (48 B.Fab user hide)
   (49 F.Fab user)
 )
@@
   (visible_elements FFFFE77F)
   (pcbplotparams
-    (layerselection 0x00030_ffffffff)
+    (layerselection 0x010fc_ffffffff)
     (usegerberextensions false)
     (usegerberattributes true)
@@
     (outputformat 1)
     (mirror false)
-    (drillshape 1)
+    (drillshape 0)
     (scaleselection 1)
     (outputdirectory ""))
@@
     (tags "QFN 0.5")
     (attr smd)
-    (fp_text reference U8 (at 2.577 3.138 180) (layer F.SilkS)
+    (fp_text reference U8 (at 3.593 -1.815 180) (layer F.SilkS)
       (effects (font (size 0.4 0.4) (thickness 0.09)))
     )
@@
     (tags "QFN 0.5")
     (attr smd)
-    (fp_text reference U9 (at 3.7465 -1.524 180) (layer F.SilkS)
+    (fp_text reference U9 (at 3.556 -1.651 180) (layer F.SilkS)
       (effects (font (size 0.4 0.4) (thickness 0.09)))
     )
@@
   (segment (start 125.222 132.727) (end 126.123 132.727) (width 0.25) (layer F.Cu) (net 1))
   (segment (start 126.123 132.727) (end 126.492 133.096) (width 0.25) (layer F.Cu) (net 1))
+  (segment (start 124.714 147.066) (end 124.714 146.431) (width 0.25) (layer B.Cu) (net 2))
+  (segment (start 124.714 146.431) (end 124.079 145.796) (width 0.25) (layer B.Cu) (net 2))
+  (via (at 124.079 145.796) (size 0.6) (drill 0.3) (layers F.Cu B.Cu) (net 2))
+  (segment (start 122.682 147.193) (end 122.682 147.066) (width 0.25) (layer F.Cu) (net 2))
+  (segment (start 122.682 147.066) (end 121.7295 146.1135) (width 0.25) (layer F.Cu) (net 2))
+  (via (at 121.7295 146.1135) (size 0.6) (drill 0.3) (layers F.Cu B.Cu) (net 2))
+  (segment (start 116.84 146.939) (end 116.84 144.5895) (width 0.25) (layer B.Cu) (net 2))
+  (segment (start 116.84 144.5895) (end 116.6495 144.399) (width 0.25) (layer B.Cu) (net 2))
+  (via (at 116.6495 144.399) (size 0.6) (drill 0.3) (layers F.Cu B.Cu) (net 2))
+  (segment (start 107.569 147.066) (end 107.569 147.701) (width 0.25) (layer F.Cu) (net 2))
+  (segment (start 107.569 147.701) (end 107.8865 148.0185) (width 0.25) (layer F.Cu) (net 2))
+  (via (at 107.8865 148.0185) (size 0.6) (drill 0.3) (layers F.Cu B.Cu) (net 2))
+  (segment (start 106.7435 149.733) (end 106.7435 148.717) (width 0.25) (layer B.Cu) (net 2))
+  (segment (start 106.7435 148.717) (end 106.4895 148.463) (width 0.25) (layer B.Cu) (net 2))
+  (via (at 106.4895 148.463) (size 0.6) (drill 0.3) (layers F.Cu B.Cu) (net 2))
+  (segment (start 105.029 150.876) (end 105.029 151.638) (width 0.25) (layer F.Cu) (net 2))
+  (segment (start 105.029 151.638) (end 104.9655 151.7015) (width 0.25) (layer F.Cu) (net 2))
+  (via (at 104.9655 151.7015) (size 0.6) (drill 0.3) (layers F.Cu B.Cu) (net 2))
+  (segment (start 105.7275 150.241) (end 105.664 150.241) (width 0.25) (layer B.Cu) (net 2))
+  (segment (start 105.664 150.241) (end 105.029 150.876) (width 0.25) (layer B.Cu) (net 2))
+  (via (at 105.029 150.876) (size 0.6) (drill 0.3) (layers F.Cu B.Cu) (net 2))
+  (segment (start 106.7435 149.733) (end 106.2355 149.733) (width 0.25) (layer F.Cu) (net 2))
+  (segment (start 106.2355 149.733) (end 105.7275 150.241) (width 0.25) (layer F.Cu) (net 2))
+  (via (at 105.7275 150.241) (size 0.6) (drill 0.3) (layers F.Cu B.Cu) (net 2))
+  (segment (start 107.7595 149.733) (end 106.7435 149.733) (width 0.25) (layer B.Cu) (net 2))
+  (via (at 106.7435 149.733) (size 0.6) (drill 0.3) (layers F.Cu B.Cu) (net 2))
+  (segment (start 109.016266 149.365234) (end 108.127266 149.365234) (width 0.25) (layer F.Cu) (net 2))
+  (segment (start 108.127266 149.365234) (end 107.7595 149.733) (width 0.25) (layer F.Cu) (net 2))
+  (via (at 107.7595 149.733) (size 0.6) (drill 0.3) (layers F.Cu B.Cu) (net 2))
+  (segment (start 109.728 149.86) (end 109.511032 149.86) (width 0.25) (layer F.Cu) (net 2))
+  (segment (start 109.511032 149.86) (end 109.016266 149.365234) (width 0.25) (layer F.Cu) (net 2))
+  (via (at 109.016266 149.365234) (size 0.6) (drill 0.3) (layers F.Cu B.Cu) (net 2))
   (segment (start 142.78475 118.84525) (end 144.68975 118.84525) (width 0.4) (layer In1.Cu) (net 2))
   (via (at 146.685 123.444) (size 0.6) (drill 0.3) (layers F.Cu B.Cu) (net 2))
